File: Eagle/src/singleBoard/twip-sb2.brd (EAGLE design)
At the start: 83.5 x 115.6 mm, 56 parts, among them J1 UJ2-BH-1-TH, Q2 IRFD9120, U1 GY-521MPU6050

Commit message: directory change
Parts:
- removed JP17, JP18: (no value), pinhead:1X01
- moved R12 10.9 mm to (21.6, 49.5), turned to 270 degrees
- moved JP16 8.98 mm to (54.6, 47.0)
- moved JP15 8.89 mm to (54.6, 72.4)
- moved Q2 4.02 mm to (27.9, 48.3)
- moved D3 3.81 mm to (41.9, 2.54)
- moved J1 2.54 mm to (52.1, 14.5)
- moved R5 2.54 mm to (31.8, 48.3)
- moved D4 1.27 mm to (59.7, 2.79)
- moved R11 1.27 mm to (34.3, 48.3)
- moved R8 1.27 mm to (39.4, 12.7)
- moved R9 1.27 mm to (59.7, 12.7)
Connections:
- removed net N$38: JP18.1, STEPDRV2.10
- removed net N$39: JP17.1, STEPDRV1.10
- new net VDD: STEPDRV1.10, STEPDRV2.10
- net N$24: now also R12.1
- net N$32: no longer R12.1
Routing:
- net N$38: track 7.40 -> 0.00 mm
- net N$39: track 5.61 -> 0.00 mm
- net N$6: track 63.0 -> 67.8 mm
- net N$24: track 5.08 -> 9.15 mm
- net N$51: track 8.89 -> 5.61 mm
- net N$29: track 101.1 -> 104.1 mm
- net N$27: track 106.2 -> 109.2 mm
- net N$32: track 45.6 -> 43.0 mm
- net N$22: track 33.2 -> 30.7 mm
- net N$30: track 12.2 -> 9.94 mm
- net N$56: track 53.7 -> 55.5 mm
- net N$48: track 64.8 -> 66.5 mm
- net N$5: track 8.15 -> 6.88 mm
- net N$23: track 34.9 -> 33.7 mm
- net N$55: track 3.81 -> 4.86 mm
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Other:
- board size 83.5 x 115.6 mm -> 83.5 x 114.3 mm
