File: Eagle/src/singleBoard/sb3.sch (EAGLE design)
At the start: 54 parts, among them J1 UJ2-BH-1-TH, Q2 IRFD9120, U1 GY-521MPU6050

Commit message: updated single board, new switches
Parts:
- removed D1, D2, D3, D4, D5: HLMP6, display-hp:HLMP6
- removed JP13, JP14: (no value), pinhead:PINHD-1X1
- removed R10, R6, R7, R8, R9: (no value), rcl:R-US_0207/10
- removed S1, S5, S6: (no value), switch:9070-1W
Connections:
- removed net N$2: C7.2, C8.2, MS2.GND, U1.ADO, U1.GND
- removed net N$52: D4.K, R9.1
- removed net N$53: D1.K, R6.1
- removed net N$54: D2.K, R7.1
- removed net N$55: D3.K, R8.1
- removed net N$57: D5.K, R10.1
- new net N$38: JP6.1
- new net N$39: SV5.4
- net N$28: no longer R10.2
- net N$31: no longer S5.S
- net N$32: no longer S6.P
- net N$36: no longer JP13.1
- net N$37: no longer JP14.1
- net N$4: no longer S5.O
- net N$40: now also J1.4, J1.SHIELD; no longer JP6.1, S6.S
- net N$41: no longer R6.2
- net N$45: no longer R7.2, S1.O
- net N$48: no longer R9.2, S1.P
- net N$56: no longer R8.2, S1.S
- net N$9: now also C7.2, C8.2, MS2.GND, U1.ADO, U1.GND; no longer D1.A, D2.A, D3.A, D4.A, D5.A, J1.4, J1.SHIELD, S5.P, SV5.4
