File: Eagle/src/singleBoard/plu/plu.brd (EAGLE design)
At the start: 99.1 x 96.6 mm, 10 parts, among them J1 5787834-2

Commit message: fix plu spacing issues found in flatcam
version P2 of PLU has a bunch of fixes to fix places where there were passages between traces, or between traces and pads that were too narrow for a 1/32 inch mill bit to pass through. 2 weren't fixable, and I added jumpers to dodge the issue. The rest of the 7 issues were resolved by small adjustments to trace locations
Parts:
- added X1, X2, X3, X4: Jmpr, con-samtec:TSW-101-XX-G-S
- CON1: value (none) -> PLU-MB-CBL
- JP1: value (none) -> PWR2MB
- JP2: value (none) -> BAT2PLU
- moved CON1 15.3 mm to (21.6, 11.4)
- moved JP1 7.73 mm to (54.6, 7.62)
- moved JP2 4.02 mm to (73.8, 7.62)
Connections:
- new net N$25: S2.3, X2.1
- new net N$28: CON1.8, X3.1
- net N$18: now also CON1.10, X1.1; no longer CON1.8, S2.3
- net N$8: now also X4.1; no longer CON1.10
Routing:
- net N$12: track 227.4 -> 170.1 mm
- net N$2: track 205.9 -> 150.5 mm
- net N$25: track 1.40 -> 34.3 mm
- net N$18: track 47.9 -> 77.5 mm
- net N$14: track 97.4 -> 124.1 mm
- net N$11: track 125.9 -> 147.5 mm
- net N$8: track 32.3 -> 12.8 mm
- net N$20: track 146.5 -> 165.1 mm
- net N$19: track 93.4 -> 81.2 mm
- net N$13: track 19.7 -> 29.4 mm
- net N$27: track 5.43 -> 14.9 mm
- net N$22: track 0.00 -> 8.89 mm
- net N$15: track 110.0 -> 101.3 mm
- net N$17: track 52.6 -> 45.6 mm
- net N$9: track 9.68 -> 16.3 mm
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