File: Eagle/src/singleBoard/sb6/sb6pads.brd (EAGLE design)
At the start: 99.1 x 96.6 mm, 31 parts, among them U1 GY-521MPU6050

Commit message: parts list, cosmetics
Parts:
- added VIA, VIA1, VIA2: (no value), pinhead:1X01
Connections:
- net 3V: now also VIA.1, VIA1.1
- net N$30: now also VIA2.1
Routing:
- net 3V: track 260.0 -> 289.3 mm
- net N$30: track 32.6 -> 53.9 mm
- net USB: track 42.3 -> 37.7 mm
- net N$4: track 110.6 -> 114.0 mm
- net N$39: track 147.2 -> 149.4 mm
- net N$9: track 76.5 -> 78.3 mm
- net N$26: track 13.3 -> 14.8 mm
- net N$33: track 511.2 -> 512.3 mm
- net N$28: track 132.1 -> 131.4 mm
- net N$23: track 17.0 -> 16.3 mm
